Commit message: Fixes SAP

File: sedna_active_perception/sedna_sap_description/urdf/asus_xtion_pro.urdf.xacro (robot description, xacro)
@@ -34,6 +34,9 @@
         <geometry>
           <!--mesh filename="xtion_pro_camera.dae"/-->
-		<box size="0.1 0.1 0.1"/>
+		<box size="0.07 0.27 0.07"/>
         </geometry>
+	<material name="black">
+		<color rgba="0.0 0.0 0.0 1"/>
+	</material>
       </visual>
       <collision>

File: sedna_active_perception/sedna_sap_description/urdf/sedna_sap.urdf.xacro (robot description, xacro)
@@ -3,9 +3,9 @@
 	<xacro:include filename="$(find sedna_description)/urdf/sedna.urdf.xacro"/>
 	<xacro:include filename="asus_xtion_pro.urdf.xacro"/>
-	<xacro:property name="cam_px" value="${body_length/2 - 0.1}" />
-    <xacro:property name="cam_py" value="0" />
+	<xacro:property name="cam_px" value="${body_length/2 - 0.01}" />
+    <xacro:property name="cam_py" value="0.02" />
         <xacro:property name="cam_pz" value="${body_height + 0.69}" />
-        <xacro:property name="cam_or" value="0" />
-        <xacro:property name="cam_op" value="0.338" />
+        <xacro:property name="cam_or" value="0.03" />
+        <xacro:property name="cam_op" value="0.339" />
         <xacro:property name="cam_oy" value="0" />
 	<xacro:sensor_asus_xtion_pro  parent="base_link"/>
