Commit message: Angst

File: sedna_active_perception/sedna_sap_description/urdf/sedna_sap.urdf.xacro (robot description, xacro)
@@ -5,7 +5,7 @@
 	<xacro:property name="cam_px" value="${body_length/2 - 0.1}" />
     <xacro:property name="cam_py" value="0" />
-        <xacro:property name="cam_pz" value="${body_height + 0.8}" />
+        <xacro:property name="cam_pz" value="${body_height + 0.69}" />
         <xacro:property name="cam_or" value="0" />
-        <xacro:property name="cam_op" value="0.3" />
+        <xacro:property name="cam_op" value="0.338" />
         <xacro:property name="cam_oy" value="0" />
 	<xacro:sensor_asus_xtion_pro  parent="base_link"/>

Commit message: Final Version

File: sedna_active_perception/sedna_sap_description/urdf/sedna_sap.urdf.xacro (robot description, xacro)
@@ -5,6 +5,6 @@
 	<xacro:property name="cam_px" value="${body_length/2 - 0.01}" />
     <xacro:property name="cam_py" value="0.02" />
-        <xacro:property name="cam_pz" value="${body_height + 0.69}" />
-        <xacro:property name="cam_or" value="0.03" />
+        <xacro:property name="cam_pz" value="${body_height + 0.66}" />
+        <xacro:property name="cam_or" value="0.0" />
         <xacro:property name="cam_op" value="0.339" />
         <xacro:property name="cam_oy" value="0" />
